File: Board Files/CT Amp.sch (EAGLE design)
At the start: 42 parts, among them IC1 LM324N

Commit message: v2 - Rerouted PCB
Original board had some problems, so I rerouted the traces
Parts:
- C1, C2, C3, C4, C5, C6: device resistor:CPOL-USE2-5 -> adafruit:CPOL-USE2.5-6
- D1, D2, D3, D4, D5, D6, D7, D8: value 1N4148DO35-10 -> IN4148; device diode:1N4148DO35-10 -> SparkFun-DiscreteSemi:DIODEPTH
- R1, R10, R11, R12, R2, R3, R4, R5, R6, R7, R8, R9: device resistor:R-US_0207/10 -> SparkFun-Resistors:RESISTORPTH-1/4W
Connections:
- net N$13: now also IC1D.OUT
- net N$21: now also IC1B.OUT
- net N$9: now also IC1C.OUT
